Commit message: Update xarm7_with_gripper.urdf

File: mani_skill2/assets/descriptions/xarm7_with_gripper.urdf (robot description, URDF)
Before this commit: robot xarm7, 18 links, 17 joints
Links:
- removed link left_inner_knuckle
- removed link right_inner_knuckle
Joints:
- removed joint left_inner_knuckle_joint
- removed joint right_inner_knuckle_joint
- joint left_finger_joint: type revolute -> fixed
- joint right_finger_joint: type revolute -> fixed
